Commit message: teleop corrected

File: rosbot_description/urdf/rosbot_core.xacro (robot description, xacro)
@@ -38,10 +38,9 @@
         <parent link="base_link"/>
         <child link="wheel_left_link"/>
-        <origin xyz="0.088 0.06100 -0.01800" rpy="0 0 0" />
-        <axis xyz="1 0 0"/>
+        <origin xyz="0.088 0.06100 -0.01800" rpy="0 1.5708 0" />
+        <axis xyz="0 0 1"/>
     </joint>
     <link name="wheel_left_link">
         <visual>
-            <origin xyz="0 0 0" rpy="0 1.5708 0"/>
             <geometry>
                 <cylinder radius="0.023" length= "0.0200"/>
@@ -52,5 +51,4 @@
         </visual>
         <collision>
-            <origin xyz="0 0 0" rpy="0 1.5708 0"/>
             <geometry>
                 <cylinder radius="0.023" length= "0.0200"/>
@@ -69,10 +67,9 @@
         <parent link="base_link"/>
         <child link="wheel_right_link"/>
-        <axis xyz="-1 0 0"/>
-        <origin rpy="0 0 0" xyz="-0.085 0.06100 -0.01750"/>
+        <axis xyz="0 0 1"/>
+        <origin rpy="0 1.5708 0" xyz="-0.085 0.06100 -0.01750"/>
     </joint>
     <link name="wheel_right_link">
         <visual>
-            <origin xyz="0 0 0" rpy="0 1.5708 0"/>
             <geometry>
                 <cylinder radius="0.023" length= "0.0200"/>
@@ -83,5 +80,4 @@
         </visual>
         <collision>
-            <origin xyz="0 0 0" rpy="0 1.5708 0"/>
             <geometry>
                 <cylinder radius="0.023" length= "0.0200"/>

File: rosbot_description/urdf/rosbot_gazebo.xacro (robot description, xacro)
@@ -47,19 +47,19 @@
           <scan>
               <horizontal>
-                  <samples>640</samples>
+                  <samples>5000</samples>
                   <resolution>1</resolution>
-                  <min_angle>-1.396263</min_angle>
-                  <max_angle>1.396263</max_angle>
+                  <min_angle>-3.14</min_angle>
+                  <max_angle>3.14</max_angle>
               </horizontal>
-              <vertical>
+              <!-- <vertical>
                   <samples>1</samples>
                   <resolution>0.01</resolution>
                   <min_angle>0</min_angle>
                   <max_angle>0</max_angle>
-              </vertical>
+              </vertical> -->
           </scan>
           <range>
-              <min>0.08</min>
-              <max>10.0</max>
+              <min>0.05</min>
+              <max>12.0</max>
               <resolution>0.01</resolution>
           </range>

Commit message: Added sensor fusion and mapping

File: rosbot_description/urdf/rosbot_core.xacro (robot description, xacro)
@@ -6,5 +6,5 @@
         <parent link="base_footprint"/>
         <child link="base_link"/>
-        <origin xyz="0 0 0.040" rpy="0 0 0"/>
+        <origin xyz="0 0 0.040" rpy="0 0 1.5708"/>
     </joint>
      <!-- Base Link -->
@@ -38,5 +38,5 @@
         <parent link="base_link"/>
         <child link="wheel_left_link"/>
-        <origin xyz="0.088 0.06100 -0.01800" rpy="0 0 0" />
+        <origin xyz="0.088 0.06100 -0.01800" rpy="0 0 0"/>
         <axis xyz="1 0 0"/>
     </joint>
@@ -45,5 +45,5 @@
             <origin xyz="0 0 0" rpy="0 1.5708 0"/>
             <geometry>
-                <cylinder radius="0.023" length= "0.0200"/>
+                <cylinder radius="0.023" length="0.0200"/>
             </geometry>
             <material name="metallic_blue">
@@ -54,5 +54,5 @@
             <origin xyz="0 0 0" rpy="0 1.5708 0"/>
             <geometry>
-                <cylinder radius="0.023" length= "0.0200"/>
+                <cylinder radius="0.023" length="0.0200"/>
             </geometry>
         </collision>
@@ -61,6 +61,6 @@
             <mass value="0.03"/>
             <inertia ixx="0.000048" ixy="0.0" ixz="0.0"
-                iyy="0.000048" iyz="0.0"
-                izz="0.0000079"/>
+                    iyy="0.000048" iyz="0.0"
+                    izz="0.0000079"/>
         </inertial>
     </link>
@@ -69,6 +69,6 @@
         <parent link="base_link"/>
         <child link="wheel_right_link"/>
-        <axis xyz="-1 0 0"/>
-        <origin rpy="0 0 0" xyz="-0.085 0.06100 -0.01750"/>
+        <origin xyz="-0.085 0.06100 -0.01750" rpy="0 0 0"/>
+        <axis xyz="1 0 0"/>
     </joint>
     <link name="wheel_right_link">
@@ -76,5 +76,5 @@
             <origin xyz="0 0 0" rpy="0 1.5708 0"/>
             <geometry>
-                <cylinder radius="0.023" length= "0.0200"/>
+                <cylinder radius="0.023" length="0.0200"/>
             </geometry>
             <material name="metallic_blue">
@@ -85,5 +85,5 @@
             <origin xyz="0 0 0" rpy="0 1.5708 0"/>
             <geometry>
-                <cylinder radius="0.023" length= "0.0200"/>
+                <cylinder radius="0.023" length="0.0200"/>
             </geometry>
         </collision>

File: rosbot_description/urdf/rosbot_gazebo.xacro (robot description, xacro)
@@ -30,41 +30,42 @@
     <maxVel>0.01</maxVel>
   </gazebo>
- <!-- ROS 2 Control -->
+  <!-- ROS 2 Control -->
+  <!-- Ignition gazebo part -->
   <gazebo>
     <plugin filename="ign_ros2_control-system" name="ign_ros2_control::IgnitionROS2ControlPlugin">
       <parameters>$(find rosbot_controller)/config/rosbot_controllers.yaml</parameters>
     </plugin>
-    <!-- inserted at the top level of the <model> tag -->
     <plugin filename="ignition-gazebo-sensors-system" name="ignition::gazebo::systems::Sensors">
         <render_engine>ogre</render_engine>
     </plugin>
   </gazebo>
+  <!-- Gazebo classic -->
+  <!-- <plugin name="gazebo_ros2_control" filename="libgazebo_ros2_control.so">
+    <robot_param>robot_description</robot_param>
+    <robot_param_node>robot_state_publisher</robot_param_node>
+    <parameters>$(find rosbot_controller)/config/rosbot_controllers.yaml</parameters>
+  </plugin> -->
   <!-- 2D Laser Sensor -->
+  <!-- Ignition Gazebo -->
   <gazebo reference="laser_link">
     <sensor name='gpu_lidar' type='gpu_lidar'>"
-      <pose relative_to='laser_link'>0 0 0 0 0 0</pose>
+      <pose relative_to='laser_link'>0 0 0.2 0 0 0</pose>
       <ray>
           <scan>
               <horizontal>
-                  <samples>640</samples>
+                  <samples>360</samples>
                   <resolution>1</resolution>
-                  <min_angle>-1.396263</min_angle>
-                  <max_angle>1.396263</max_angle>
+                  <min_angle>-3.1416</min_angle>
+                  <max_angle>3.1416</max_angle>
               </horizontal>
-              <vertical>
-                  <samples>1</samples>
-                  <resolution>0.01</resolution>
-                  <min_angle>0</min_angle>
-                  <max_angle>0</max_angle>
-              </vertical>
           </scan>
           <range>
-              <min>0.08</min>
-              <max>10.0</max>
+              <min>0.25</min>
+              <max>8.0</max>
               <resolution>0.01</resolution>
           </range>
       </ray>
       <always_on>1</always_on>
-      <update_rate>30</update_rate>
+      <update_rate>10</update_rate>
       <visualize>true</visualize>
       <topic>/scan</topic>
@@ -73,3 +74,31 @@
     </sensor>
   </gazebo>
+  <!-- Gazebo classic -->
+  <!-- <gazebo reference="laser_link">
+    <sensor name="lidar" type="ray">
+      <pose>0 0 0 0 0 0</pose>
+      <ray>
+        <scan>
+          <horizontal>
+            <samples>500</samples>
+            <resolution>1</resolution>
+            <min_angle>-3.14</min_angle>
+            <max_angle>3.14</max_angle>
+          </horizontal>
+        </scan>
+        <range>
+          <min>0.05</min>
+          <max>12.0</max>
+          <resolution>0.01</resolution>
+        </range>
+      </ray>
+      <always_on>true</always_on>
+      <update_rate>30</update_rate>
+      <visualize>true</visualize>
+      <plugin name="gazebo_ros_laser_controller" filename="libgazebo_ros_ray_sensor.so">
+        <topicName>/scan</topicName>
+        <frameName>laser_link</frameName>
+      </plugin>
+    </sensor>
+  </gazebo>  -->
 </robot>

File: rosbot_description/urdf/rosbot_imu.xacro (robot description, xacro)
@@ -5,7 +5,8 @@
         <parent link="base_link"/>
         <child link="imu_link"/>
-        <origin xyz="0.0 0 0.068" rpy="0 0 0"/>
+        <origin xyz="0.0 0 0.040" rpy="0 0 -1.5708"/>
     </joint>
     <link name="imu_link"/>
+    <!-- Ignition Gazebo -->
     <gazebo reference="imu_link">
         <sensor name="imu_sensor" type="imu">
@@ -72,3 +73,16 @@
         </sensor>
     </gazebo>
+    <!-- Gazebo Classic -->
+    <!-- <gazebo reference="imu_link">
+        <sensor name="imu_sensor" type="imu">
+            <pose>0 0 0 0 0 0</pose>
+            <always_on>true</always_on>
+            <update_rate>100</update_rate>
+            <visualize>true</visualize>
+            <plugin name="imu_plugin" filename="libgazebo_ros_imu_sensor.so">
+            <topicName>imu</topicName>
+            <frameName>imu_link</frameName>
+            </plugin>
+        </sensor>
+    </gazebo> -->
 </robot>

File: rosbot_description/urdf/rosbot_lidar.xacro (robot description, xacro)
@@ -4,5 +4,5 @@
         <parent link="base_link"/>
         <child link="laser_link"/>
-        <origin xyz="0 0 0.125" rpy="0 0 0"/>
+        <origin xyz="0 0 0.125" rpy="0 0 -1.5708"/>
     </joint>
     <link name="laser_link">

File: rosbot_description/urdf/rosbot_ros2_control.xacro (robot description, xacro)
@@ -2,6 +2,8 @@
 <robot xmlns:xacro="http://www.ros.org/wiki/xacro" name="rosbot">
     <ros2_control name="IgnitionSystem" type="system">
+    <!-- <ros2_control name="GazeboSystem" type="system"> -->
         <hardware>
             <plugin>ign_ros2_control/IgnitionSystem</plugin>
+            <!-- <plugin>gazebo_ros2_control/GazeboSystem</plugin> -->
         </hardware>
         <!-- ros2_control Common Interfaces -->
